Commit message: Added diff drive, fixed wheel axis

File: src/igv_assembly/urdf/igv_assembly.urdf (robot description, URDF)
Before this commit: robot igv_assembly, 13 links, 12 joints
Joints:
- joint WL1: axis 0 -1 0 -> 0 1 0
- joint WL2: axis 0 -1 0 -> 0 1 0
- joint WL3: axis 0 -1 0 -> 0 1 0

Commit message: Akshit is gay only for Yash

File: src/igv_assembly/urdf/igv_assembly.urdf (robot description, URDF)
Before this commit: robot igv_assembly, 13 links, 12 joints
Links:
- added link DepthCamOptical
- added link DepthCamVirtual
- link DepthCam: mass 0.213055140920182 -> 0.01
- link RockerL: mass 0.0957401232694818 -> 0.118438130191668
- link RockerR: mass 0.0975809423226696 -> 0.120278949244856
- link WheelR1: mass 0.095683487480657 -> 0.0956834874806569
- link base_link: mass 1.55304637865748 -> 1.50765036481311
Joints:
- added joint depth_cam_virtual_joint: type fixed, parent DepthCam, child DepthCamVirtual, origin xyz=0.05 0 0 rpy=0 0 0
- added joint optical_joint: type fixed, parent DepthCamVirtual, child DepthCamOptical, origin xyz=0 0 0 rpy=-1.5708 0 -1.5708
- joint DC: axis 0 -1 0 -> 0 1 0; type continuous -> fixed
- joint DC_Base: origin xyz=-0.005 0.255 0.075 rpy=0 0 0 -> xyz=0.169117512201439 0 0.0874999999999999 rpy=0 0 0
- joint LeftBogie: axis 0 -1 0 -> 0 1 0; origin xyz=-0.111132840749356 -0.0165000000000001 -0.0391246943371841 rpy=0 0 0 -> xyz=0.111132840749356 0.0165000000000001 -0.0391246943371841 rpy=0 0 0
- joint LeftRocker: axis 0 -1 0 -> 0 1 0; limit lower=-0.5236 upper=0.5236 effort=100 velocity=1 -> (none); origin xyz=0.155 -0.048123 0.065 rpy=0 0 0 -> xyz=0 0.203122560056477 0.0550000000000017 rpy=0 0 0; type revolute -> fixed
- joint RightBogie: axis 0 -1 0 -> 0 1 0; origin xyz=-0.10945532574041 -0.00200000000000045 -0.0519690452775528 rpy=0 0 0 -> xyz=0.10945532574041 0.00200000000000045 -0.0519690452775528 rpy=0 0 0
- joint RightRocker: axis 0 -1 0 -> 0 1 0; limit lower=-0.5236 upper=0.5236 effort=100 velocity=1 -> (none); origin xyz=0.155 0.35504 0.075 rpy=0 0 0 -> xyz=0 -0.200038955864052 0.0649999999999993 rpy=0 0 0; type revolute -> fixed
- joint WL1: origin xyz=-0.118211585773428 -0.046 -0.0768587730121344 rpy=0 0 0 -> xyz=0.118211585773428 0.046 -0.0768587730121344 rpy=0 0 0
- joint WL2: origin xyz=0.106228768769022 -0.046 -0.0927183837532437 rpy=0 0 0 -> xyz=-0.106228768769022 0.046 -0.0927183837532437 rpy=0 0 0
- joint WL3: origin xyz=0.229272035427498 -0.0495 -0.111621385813536 rpy=0 0 0 -> xyz=-0.229272035427498 0.0495 -0.111621385813536 rpy=0 0 0
- joint WR1: origin xyz=-0.122211174343328 0.0660000000000005 -0.0703255207277187 rpy=0 0 0 -> xyz=0.122211174343328 -0.0660000000000005 -0.0703255207277187 rpy=0 0 0
- joint WR2: origin xyz=0.101036656375721 0.0700000000000005 -0.0983506180377884 rpy=0 0 0 -> xyz=-0.101036656375721 -0.0700000000000005 -0.0983506180377884 rpy=0 0 0
- joint WR3: origin xyz=0.232712347234891 0.048 -0.115628558083324 rpy=0 0 0 -> xyz=-0.232712347234891 -0.048 -0.115628558083324 rpy=0 0 0
