Commit message: I commited I swear

File: src/igv_assembly/urdf/simple_bot.urdf.xacro (robot description, xacro)
@@ -18,5 +18,5 @@
   <link name="FL_Wheel">
     <visual><geometry><cylinder radius="0.1" length="0.05"/></geometry></visual>
-    <collision><geometry><cylinder radius="0.1" length="0.05"/></geometry></collision>
+    <collision><geometry><sphere radius="0.1"/></geometry></collision>
     <inertial><mass value="1.0"/><inertia ixx="0.003" ixy="0" ixz="0" iyy="0.003" iyz="0" izz="0.005"/></inertial>
   </link>
@@ -29,5 +29,5 @@
   <link name="FR_Wheel">
     <visual><geometry><cylinder radius="0.1" length="0.05"/></geometry></visual>
-    <collision><geometry><cylinder radius="0.1" length="0.05"/></geometry></collision>
+    <collision><geometry><sphere radius="0.1"/></geometry></collision>
     <inertial><mass value="1.0"/><inertia ixx="0.003" ixy="0" ixz="0" iyy="0.003" iyz="0" izz="0.005"/></inertial>
   </link>
@@ -40,5 +40,5 @@
   <link name="RL_Wheel">
     <visual><geometry><cylinder radius="0.1" length="0.05"/></geometry></visual>
-    <collision><geometry><cylinder radius="0.1" length="0.05"/></geometry></collision>
+    <collision><geometry><sphere radius="0.1"/></geometry></collision>
     <inertial><mass value="1.0"/><inertia ixx="0.003" ixy="0" ixz="0" iyy="0.003" iyz="0" izz="0.005"/></inertial>
   </link>
@@ -51,5 +51,5 @@
   <link name="RR_Wheel">
     <visual><geometry><cylinder radius="0.1" length="0.05"/></geometry></visual>
-    <collision><geometry><cylinder radius="0.1" length="0.05"/></geometry></collision>
+    <collision><geometry><sphere radius="0.1"/></geometry></collision>
     <inertial><mass value="1.0"/><inertia ixx="0.003" ixy="0" ixz="0" iyy="0.003" iyz="0" izz="0.005"/></inertial>
   </link>
@@ -126,29 +126,33 @@
   <gazebo reference="FL_Wheel">
     <mu1>1.0</mu1>
-    <mu2>0.1</mu2>
-    <kp>10000000.0</kp>
-    <kd>1.0</kd>
+    <mu2>0.2</mu2>
+    <kp>100000.0</kp>
+    <kd>100.0</kd>
     <minDepth>0.001</minDepth>
+    <fdir1>1 0 0</fdir1>
   </gazebo>
   <gazebo reference="FR_Wheel">
     <mu1>1.0</mu1>
-    <mu2>0.1</mu2>
-    <kp>10000000.0</kp>
-    <kd>1.0</kd>
+    <mu2>0.2</mu2>
+    <kp>100000.0</kp>
+    <kd>100.0</kd>
     <minDepth>0.001</minDepth>
+    <fdir1>1 0 0</fdir1>
   </gazebo>
   <gazebo reference="RL_Wheel">
     <mu1>1.0</mu1>
-    <mu2>0.1</mu2>
-    <kp>10000000.0</kp>
-    <kd>1.0</kd>
+    <mu2>0.2</mu2>
+    <kp>100000.0</kp>
+    <kd>100.0</kd>
     <minDepth>0.001</minDepth>
+    <fdir1>1 0 0</fdir1>
   </gazebo>
   <gazebo reference="RR_Wheel">
     <mu1>1.0</mu1>
-    <mu2>0.1</mu2>
-    <kp>10000000.0</kp>
-    <kd>1.0</kd>
+    <mu2>0.2</mu2>
+    <kp>100000.0</kp>
+    <kd>100.0</kd>
     <minDepth>0.001</minDepth>
+    <fdir1>1 0 0</fdir1>
   </gazebo>
 </robot>

Commit message: Odom fixed Rtab kinda working

File: src/igv_assembly/urdf/simple_bot.urdf.xacro (robot description, xacro)
@@ -1,5 +1,5 @@
 <?xml version="1.0"?>
 <robot name="simple_bot" xmlns:xacro="http://www.ros.org/wiki/xacro">
-  <!-- ================= CHASSIS ================= -->
+  <!-- ================= BASE LINK ================= -->
   <link name="base_link">
     <visual>
@@ -15,49 +15,40 @@
     </inertial>
   </link>
-  <!-- ================= WHEELS ================= -->
-  <link name="FL_Wheel">
-    <visual><geometry><cylinder radius="0.1" length="0.05"/></geometry></visual>
-    <collision><geometry><sphere radius="0.1"/></geometry></collision>
-    <inertial><mass value="1.0"/><inertia ixx="0.003" ixy="0" ixz="0" iyy="0.003" iyz="0" izz="0.005"/></inertial>
-  </link>
-  <joint name="FL_Joint" type="continuous">
-    <parent link="base_link"/>
-    <child link="FL_Wheel"/>
-    <origin xyz="0.15 0.15 0" rpy="-1.5708 0 0"/>
-    <axis xyz="0 0 1"/>
-  </joint>
-  <link name="FR_Wheel">
-    <visual><geometry><cylinder radius="0.1" length="0.05"/></geometry></visual>
-    <collision><geometry><sphere radius="0.1"/></geometry></collision>
-    <inertial><mass value="1.0"/><inertia ixx="0.003" ixy="0" ixz="0" iyy="0.003" iyz="0" izz="0.005"/></inertial>
-  </link>
-  <joint name="FR_Joint" type="continuous">
-    <parent link="base_link"/>
-    <child link="FR_Wheel"/>
-    <origin xyz="0.15 -0.15 0" rpy="-1.5708 0 0"/>
-    <axis xyz="0 0 1"/>
-  </joint>
-  <link name="RL_Wheel">
-    <visual><geometry><cylinder radius="0.1" length="0.05"/></geometry></visual>
-    <collision><geometry><sphere radius="0.1"/></geometry></collision>
-    <inertial><mass value="1.0"/><inertia ixx="0.003" ixy="0" ixz="0" iyy="0.003" iyz="0" izz="0.005"/></inertial>
-  </link>
-  <joint name="RL_Joint" type="continuous">
-    <parent link="base_link"/>
-    <child link="RL_Wheel"/>
-    <origin xyz="-0.15 0.15 0" rpy="-1.5708 0 0"/>
-    <axis xyz="0 0 1"/>
-  </joint>
-  <link name="RR_Wheel">
-    <visual><geometry><cylinder radius="0.1" length="0.05"/></geometry></visual>
-    <collision><geometry><sphere radius="0.1"/></geometry></collision>
-    <inertial><mass value="1.0"/><inertia ixx="0.003" ixy="0" ixz="0" iyy="0.003" iyz="0" izz="0.005"/></inertial>
-  </link>
-  <joint name="RR_Joint" type="continuous">
-    <parent link="base_link"/>
-    <child link="RR_Wheel"/>
-    <origin xyz="-0.15 -0.15 0" rpy="-1.5708 0 0"/>
-    <axis xyz="0 0 1"/>
-  </joint>
+  <!-- ================= WHEEL MACRO ================= -->
+<!-- ================= WHEEL MACRO ================= -->
+  <xacro:macro name="wheel" params="prefix x_reflect y_reflect">
+    <link name="${prefix}_Wheel">
+      <visual>
+        <geometry><cylinder radius="0.1" length="0.05"/></geometry>
+      </visual>
+      <collision>
+        <geometry><sphere radius="0.1"/></geometry>
+      </collision>
+      <inertial>
+        <mass value="1.0"/>
+        <inertia ixx="0.003" ixy="0" ixz="0" iyy="0.003" iyz="0" izz="0.005"/>
+      </inertial>
+    </link>
+    <joint name="${prefix}_Joint" type="continuous">
+      <parent link="base_link"/>
+      <child link="${prefix}_Wheel"/>
+      <origin xyz="${x_reflect * 0.15} ${y_reflect * 0.15} 0" rpy="-1.5708 0 0"/>
+      <axis xyz="0 0 1"/>
+    </joint>
+    <gazebo reference="${prefix}_Wheel">
+      <mu1>1.0</mu1>
+      <mu2>0.2</mu2>
+      <!-- fdir1 locks the high friction to the wheel's local X axis (forward) -->
+      <fdir1>1 0 0</fdir1>
+      <!-- Increased kp makes the wheels solid so the chassis stops sagging and scraping -->
+      <kp>10000000.0</kp>
+      <kd>1.0</kd>
+      <minDepth>0.001</minDepth>
+    </gazebo>
+  </xacro:macro>
+  <xacro:wheel prefix="FL" x_reflect="1"  y_reflect="1" />
+  <xacro:wheel prefix="FR" x_reflect="1"  y_reflect="-1" />
+  <xacro:wheel prefix="RL" x_reflect="-1" y_reflect="1" />
+  <xacro:wheel prefix="RR" x_reflect="-1" y_reflect="-1" />
   <!-- ================= CAMERA ================= -->
   <link name="DepthCamVirtual">
@@ -75,13 +66,6 @@
     <origin xyz="0 0 0" rpy="-1.5708 0 -1.5708"/>
   </joint>
-  <!-- ================= GAZEBO PHYSICS & PLUGINS ================= -->
-  <gazebo reference="FL_Wheel"><mu1>1.0</mu1><mu2>0.1</mu2><minDepth>0.001</minDepth></gazebo>
-  <gazebo reference="FR_Wheel"><mu1>1.0</mu1><mu2>0.1</mu2><minDepth>0.001</minDepth></gazebo>
-  <gazebo reference="RL_Wheel"><mu1>1.0</mu1><mu2>0.1</mu2><minDepth>0.001</minDepth></gazebo>
-  <gazebo reference="RR_Wheel"><mu1>1.0</mu1><mu2>0.1</mu2><minDepth>0.001</minDepth></gazebo>
+  <!-- ================= GAZEBO SENSORS & CONTROL ================= -->
   <gazebo>
-    <plugin filename="gz-sim-joint-state-publisher-system" name="gz::sim::systems::JointStatePublisher">
-      <topic>joint_states</topic>
-    </plugin>
     <plugin filename="gz_ros2_control-system" name="gz_ros2_control::GazeboSimROS2ControlPlugin">
       <parameters>$(find igv_assembly)/config/simple_controllers.yaml</parameters>
@@ -94,65 +78,35 @@
     <sensor type='rgbd_camera' name="Depth_Camera">
       <always_on>true</always_on>
-      <update_rate>15.0</update_rate>
+      <update_rate>30.0</update_rate>
       <topic>depth_camera</topic>
       <camera name="depth_camera">
         <optical_frame_id>DepthCamOptical</optical_frame_id>
-        <horizontal_fov>1.777</horizontal_fov>
-        <image><width>1280</width><height>720</height><format>R8G8B8</format></image>
+        <horizontal_fov>1.047</horizontal_fov>
+        <image><width>640</width><height>480</height><format>R8G8B8</format></image>
         <clip><near>0.1</near><far>10.0</far></clip>
       </camera>
     </sensor>
   </gazebo>
-  <!-- ================= ROS2 CONTROL ================= -->
+  <!-- ================= ROS 2 CONTROL HARDWARE ================= -->
   <ros2_control name="IgnitionSystem" type="system">
-      <hardware><plugin>gz_ros2_control/GazeboSimSystem</plugin></hardware>
-      <joint name="FL_Joint">
-        <command_interface name="velocity"/>
-        <state_interface name="position"/><state_interface name="velocity"/>
-      </joint>
-      <joint name="FR_Joint">
-        <command_interface name="velocity"/>
-        <state_interface name="position"/><state_interface name="velocity"/>
-      </joint>
-      <joint name="RL_Joint">
-        <command_interface name="velocity"/>
-        <state_interface name="position"/><state_interface name="velocity"/>
-      </joint>
-      <joint name="RR_Joint">
-        <command_interface name="velocity"/>
-        <state_interface name="position"/><state_interface name="velocity"/>
-      </joint>
+    <hardware>
+      <plugin>gz_ros2_control/GazeboSimSystem</plugin>
+    </hardware>
+    <joint name="FL_Joint">
+      <command_interface name="velocity"/>
+      <state_interface name="position"/><state_interface name="velocity"/>
+    </joint>
+    <joint name="FR_Joint">
+      <command_interface name="velocity"/>
+      <state_interface name="position"/><state_interface name="velocity"/>
+    </joint>
+    <joint name="RL_Joint">
+      <command_interface name="velocity"/>
+      <state_interface name="position"/><state_interface name="velocity"/>
+    </joint>
+    <joint name="RR_Joint">
+      <command_interface name="velocity"/>
+      <state_interface name="position"/><state_interface name="velocity"/>
+    </joint>
   </ros2_control>
-  <gazebo reference="FL_Wheel">
-    <mu1>1.0</mu1>
-    <mu2>0.2</mu2>
-    <kp>100000.0</kp>
-    <kd>100.0</kd>
-    <minDepth>0.001</minDepth>
-    <fdir1>1 0 0</fdir1>
-  </gazebo>
-  <gazebo reference="FR_Wheel">
-    <mu1>1.0</mu1>
-    <mu2>0.2</mu2>
-    <kp>100000.0</kp>
-    <kd>100.0</kd>
-    <minDepth>0.001</minDepth>
-    <fdir1>1 0 0</fdir1>
-  </gazebo>
-  <gazebo reference="RL_Wheel">
-    <mu1>1.0</mu1>
-    <mu2>0.2</mu2>
-    <kp>100000.0</kp>
-    <kd>100.0</kd>
-    <minDepth>0.001</minDepth>
-    <fdir1>1 0 0</fdir1>
-  </gazebo>
-  <gazebo reference="RR_Wheel">
-    <mu1>1.0</mu1>
-    <mu2>0.2</mu2>
-    <kp>100000.0</kp>
-    <kd>100.0</kd>
-    <minDepth>0.001</minDepth>
-    <fdir1>1 0 0</fdir1>
-  </gazebo>
 </robot>
