Commit message: Changed params

File: src/igv_assembly/urdf/igv_assembly.urdf.xacro (robot description, xacro)
@@ -4,5 +4,5 @@
      For more information, please see http://wiki.ros.org/sw_urdf_exporter -->
 <robot
-  name="igv_assembly">
+  name="igv_assembly" xmlns:xacro="http://www.ros.org/wiki/xacro">
   <link
     name="base_link">
@@ -706,34 +706,14 @@
     </joint>
   <gazebo>
-  <!-- <plugin filename="ignition-gazebo-diff-drive-system" name="ignition::gazebo::systems::DiffDrive">
-      <left_joint>WL1</left_joint>
-      <left_joint>WL2</left_joint>
-      <left_joint>WL3</left_joint>
-      <right_joint>WR1</right_joint>
-      <right_joint>WR2</right_joint>
-      <right_joint>WR3</right_joint>
-      <wheel_separation>0.550</wheel_separation>
-      <wheel_radius>0.100</wheel_radius>
-      <odom_publish_frequency>50</odom_publish_frequency>
-      <odom_topic>odom</odom_topic>
-      <topic>cmd_vel</topic>
-      <frame_id>odom</frame_id>
-      <child_frame_id>base_link</child_frame_id>
-      <tf_topic>/tf</tf_topic>
-  </plugin> -->
-  <plugin filename="ignition-gazebo-joint-state-publisher-system" name="ignition::gazebo::systems::JointStatePublisher">
-  <topic>joint_states</topic>
-  </plugin>
-  <plugin filename="ign_ros2_control-system" name="ign_ros2_control::IgnitionROS2ControlPlugin">
-    <parameters>$(find igv_assembly)/config/controllers.yaml</parameters>
-  </plugin>
-  <plugin
-      filename="ignition-gazebo-sensors-system"
-      name="ignition::gazebo::systems::Sensors">
+    <plugin filename="gz-sim-joint-state-publisher-system" name="gz::sim::systems::JointStatePublisher">
+      <topic>joint_states</topic>
+    </plugin>
+    <plugin filename="gz_ros2_control-system" name="gz_ros2_control::GazeboSimROS2ControlPlugin">
+      <parameters>$(find igv_assembly)/config/controllers.yaml</parameters>
+    </plugin>
+    <plugin filename="gz-sim-sensors-system" name="gz::sim::systems::Sensors">
       <render_engine>ogre2</render_engine>
     </plugin>
-    <plugin
-      filename="ignition-gazebo-imu-system"
-      name="ignition::gazebo::systems::Imu">
+    <plugin filename="gz-sim-imu-system" name="gz::sim::systems::Imu">
     </plugin>
   </gazebo>
@@ -752,10 +732,6 @@
         </image>
         <clip>
-            <near>
-              0.1
-            </near>
-            <far>
-              10.0
-            </far>
+          <near>0.1</near>
+          <far>10.0</far>
         </clip>
         <lens>
@@ -773,6 +749,12 @@
   <ros2_control name="IgnitionSystem" type="system">
       <hardware>
-        <plugin>ign_ros2_control/IgnitionSystem</plugin>
+        <plugin>gz_ros2_control/GazeboSimSystem</plugin>
       </hardware>
+      <joint name="RightBogie">
+        <state_interface name="position"/>
+      </joint>
+      <joint name="LeftBogie">
+        <state_interface name="position"/>
+      </joint>
       <joint name="WL1">
         <command_interface name="velocity">

Commit message: NAVYA IS THE BEST PERSON

File: src/igv_assembly/urdf/igv_assembly.urdf.xacro (robot description, xacro)
@@ -3,694 +3,374 @@
      Commit Version: 1.6.0-4-g7f85cfe  Build Version: 1.6.7995.38578
      For more information, please see http://wiki.ros.org/sw_urdf_exporter -->
-<robot
-  name="igv_assembly" xmlns:xacro="http://www.ros.org/wiki/xacro">
-  <link
-    name="base_link">
-    <inertial>
-      <origin
-        xyz="-5.55111512312578E-16 4.44089209850063E-16 0.0131058382964258"
-        rpy="0 0 0" />
-      <mass
-        value="1.50765036481311" />
-      <inertia
-        ixx="0.0172819216111337"
-        ixy="-4.34830427033138E-18"
-        ixz="-1.39771001490249E-18"
-        iyy="0.0174462077143803"
-        iyz="-5.3897948963004E-06"
-        izz="0.0322556766841891" />
-    </inertial>
-    <visual>
-      <origin
-        xyz="0 0 0"
-        rpy="0 0 0" />
-      <geometry>
-        <mesh
-          filename="package://igv_assembly/meshes/base_link.STL" />
-      </geometry>
-      <material
-        name="">
-        <color
-          rgba="0.627450980392157 0.627450980392157 0.627450980392157 1" />
-      </material>
-    </visual>
-    <collision>
-      <origin
-        xyz="0 0 0"
-        rpy="0 0 0" />
-      <geometry>
-        <mesh
-          filename="package://igv_assembly/meshes/base_link.STL" />
-      </geometry>
-    </collision>
-  </link>
-  <link
-    name="RockerL">
-    <inertial>
-      <origin
-        xyz="-0.0444283900462424 -0.00756705252802037 -0.0391939612078949"
-        rpy="0 0 0" />
-      <mass
-        value="0.118438130191668" />
-      <inertia
-        ixx="0.000155017015084251"
-        ixy="-1.48646750943822E-21"
-        ixz="-0.000283635186660913"
-        iyy="0.00115834975412409"
-        iyz="3.29563792754343E-22"
-        izz="0.0010417268635807" />
-    </inertial>
-    <visual>
-      <origin
-        xyz="0 0 0"
-        rpy="0 0 0" />
-      <geometry>
-        <mesh
-          filename="package://igv_assembly/meshes/RockerL.STL" />
-      </geometry>
-      <material
-        name="">
-        <color
-          rgba="0.627450980392157 0.627450980392157 0.627450980392157 1" />
-      </material>
-    </visual>
-    <collision>
-      <origin
-        xyz="0 0 0"
-        rpy="0 0 0" />
-      <geometry>
-        <mesh
-          filename="package://igv_assembly/meshes/RockerL.STL" />
-      </geometry>
-    </collision>
-  </link>
-  <joint
-    name="LeftRocker"
-    type="fixed">
-    <origin
-      xyz="0 0.203122560056477 0.0550000000000017"
-      rpy="0 0 0" />
-    <parent
-      link="base_link" />
-    <child
-      link="RockerL" />
-    <axis
-      xyz="0 1 0" />
-  </joint>
-  <link
-    name="WheelL3">
-    <inertial>
-      <origin
-        xyz="0 -0.0165713300799556 2.22044604925031E-16"
-        rpy="0 0 0" />
-      <mass
-        value="0.095683487480657" />
-      <inertia
-        ixx="9.61942691845856E-05"
-        ixy="-2.67115443245389E-20"
-        ixz="4.67357046092461E-20"
-        iyy="0.000167342984972362"
-        iyz="2.38694734300935E-20"
-        izz="9.61942691845857E-05" />
-    </inertial>
-    <visual>
-      <origin
-        xyz="0 0 0"
-        rpy="0 0 0" />
-      <geometry>
-        <mesh
-          filename="package://igv_assembly/meshes/WheelL3.STL" />
-      </geometry>
-      <material
-        name="">
-        <color
-          rgba="0.627450980392157 0.627450980392157 0.627450980392157 1" />
-      </material>
-    </visual>
-    <collision>
-      <origin
-        xyz="0 0 0"
-        rpy="0 0 0" />
-      <geometry>
-        <mesh
-          filename="package://igv_assembly/meshes/WheelL3.STL" />
-      </geometry>
-    </collision>
-  </link>
-  <joint
-    name="WL3"
-    type="continuous">
-    <origin
-      xyz="-0.229272035427498 0.0495 -0.111621385813536"
-      rpy="0 0 0" />
-    <parent
-      link="RockerL" />
-    <child
-      link="WheelL3" />
-    <axis
-      xyz="0 1 0" />
-  </joint>
-  <link
-    name="BogieL">
-    <inertial>
-      <origin
-        xyz="0.00360601465125077 -0.00199999999999989 -0.0510312150797347"
-        rpy="0 0 0" />
-      <mass
-        value="0.0725855377820986" />
-      <inertia
-        ixx="8.05328649275476E-05"
-        ixy="-1.61236687743738E-21"
-        ixz="-2.47858215964137E-05"
-        iyy="0.000509872951246973"
-        iyz="1.43622722355043E-21"
-        izz="0.000429542783513456" />
-    </inertial>
-    <visual>
-      <origin
-        xyz="0 0 0"
-        rpy="0 0 0" />
-      <geometry>
-        <mesh
-          filename="package://igv_assembly/meshes/BogieL.STL" />
-      </geometry>
-      <material
-        name="">
-        <color
-          rgba="0.752941176470588 0.752941176470588 0.752941176470588 1" />
-      </material>
-    </visual>
-    <collision>
-      <origin
-        xyz="0 0 0"
-        rpy="0 0 0" />
-      <geometry>
-        <mesh
-          filename="package://igv_assembly/meshes/BogieL.STL" />
-      </geometry>
-    </collision>
-  </link>
-  <joint
-    name="LeftBogie"
-    type="revolute">
-    <origin
-      xyz="0.111132840749356 0.0165000000000001 -0.0391246943371841"
-      rpy="0 0 0" />
-    <parent
-      link="RockerL" />
-    <child
-      link="BogieL" />
-    <axis
-      xyz="0 1 0" />
-    <limit
-      lower="-0.2618"
-      upper="0.2618"
-      effort="100"
-      velocity="1" />
-  </joint>
-  <link
-    name="WheelL2">
-    <inertial>
-      <origin
-        xyz="0 -0.0165713300799556 0"
-        rpy="0 0 0" />
-      <mass
-        value="0.095683487480657" />
-      <inertia
-        ixx="9.61942691845856E-05"
-        ixy="-3.36416595964494E-20"
-        ixz="4.94771621050058E-20"
-        iyy="0.000167342984972362"
-        iyz="3.33241050522677E-20"
-        izz="9.61942691845857E-05" />
-    </inertial>
-    <visual>
-      <origin
-        xyz="0 0 0"
-        rpy="0 0 0" />
-      <geometry>
-        <mesh
-          filename="package://igv_assembly/meshes/WheelL2.STL" />
-      </geometry>
-      <material
-        name="">
-        <color
-          rgba="0.627450980392157 0.627450980392157 0.627450980392157 1" />
-      </material>
-    </visual>
-    <collision>
-      <origin
-        xyz="0 0 0"
-        rpy="0 0 0" />
-      <geometry>
-        <mesh
-          filename="package://igv_assembly/meshes/WheelL2.STL" />
-      </geometry>
-    </collision>
-  </link>
-  <joint
-    name="WL2"
-    type="continuous">
-    <origin
-      xyz="-0.106228768769022 0.046 -0.0927183837532437"
-      rpy="0 0 0" />
-    <parent
-      link="BogieL" />
-    <child
-      link="WheelL2" />
-    <axis
-      xyz="0 1 0" />
-  </joint>
-  <link
-    name="WheelL1">
-    <inertial>
-      <origin
-        xyz="0 -0.0165713300799556 0"
-        rpy="0 0 0" />
-      <mass
-        value="0.095683487480657" />
-      <inertia
-        ixx="9.61942691845857E-05"
-        ixy="-1.84881341438237E-20"
-        ixz="4.73560900686608E-20"
-        iyy="0.000167342984972362"
-        iyz="2.65291537628972E-20"
-        izz="9.61942691845858E-05" />
-    </inertial>
-    <visual>
-      <origin
-        xyz="0 0 0"
-        rpy="0 0 0" />
-      <geometry>
-        <mesh
-          filename="package://igv_assembly/meshes/WheelL1.STL" />
-      </geometry>
-      <material
-        name="">
-        <color
-          rgba="0.627450980392157 0.627450980392157 0.627450980392157 1" />
-      </material>
-    </visual>
-    <collision>
-      <origin
-        xyz="0 0 0"
-        rpy="0 0 0" />
-      <geometry>
-        <mesh
-          filename="package://igv_assembly/meshes/WheelL1.STL" />
-      </geometry>
-    </collision>
-  </link>
-  <joint
-    name="WL1"
-    type="continuous">
-    <origin
-      xyz="0.118211585773428 0.046 -0.0768587730121344"
-      rpy="0 0 0" />
-    <parent
-      link="BogieL" />
-    <child
-      link="WheelL1" />
-    <axis
-      xyz="0 1 0" />
-  </joint>
-  <link
-    name="RockerR">
-    <inertial>
-      <origin
-        xyz="-0.0458474111089989 0.00875620819604439 -0.0427777170935231"
-        rpy="0 0 0" />
-      <mass
-        value="0.120278949244856" />
-      <inertia
-        ixx="0.000159183946373948"
-        ixy="6.14879409715585E-22"
-        ixz="-0.000276551948895894"
-        iyy="0.00119888716107189"
-        iyz="-6.87470951019029E-22"
-        izz="0.0010781022480896" />
-    </inertial>
-    <visual>
-      <origin
-        xyz="0 0 0"
-        rpy="0 0 0" />
-      <geometry>
-        <mesh
-          filename="package://igv_assembly/meshes/RockerR.STL" />
-      </geometry>
-      <material
-        name="">
-        <color
-          rgba="0.627450980392157 0.627450980392157 0.627450980392157 1" />
-      </material>
-    </visual>
-    <collision>
-      <origin
-        xyz="0 0 0"
-        rpy="0 0 0" />
-      <geometry>
-        <mesh
-          filename="package://igv_assembly/meshes/RockerR.STL" />
-      </geometry>
-    </collision>
-  </link>
-  <joint
-    name="RightRocker"
-    type="fixed">
-    <origin
-      xyz="0 -0.200038955864052 0.0649999999999993"
-      rpy="0 0 0" />
-    <parent
-      link="base_link" />
-    <child
-      link="RockerR" />
-    <axis
-      xyz="0 1 0" />
-  </joint>
-  <link
-    name="WheelR3">
-    <inertial>
-      <origin
-        xyz="0 0.0165713300799555 0"
-        rpy="0 0 0" />
-      <mass
-        value="0.095683487480657" />
-      <inertia
-        ixx="9.61942691845858E-05"
-        ixy="2.29863529225909E-20"
-        ixz="5.32512598144256E-21"
-        iyy="0.000167342984972362"
-        iyz="-6.37858672378045E-21"
-        izz="9.61942691845856E-05" />
-    </inertial>
-    <visual>
-      <origin
-        xyz="0 0 0"
-        rpy="0 0 0" />
-      <geometry>
-        <mesh
-          filename="package://igv_assembly/meshes/WheelR3.STL" />
-      </geometry>
-      <material
-        name="">
-        <color
-          rgba="0.627450980392157 0.627450980392157 0.627450980392157 1" />
-      </material>
-    </visual>
-    <collision>
-      <origin
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